File: schematic/NixieClock.sch (KiCad schematic (older format))
At the start: 22 parts

Commit message: Small changes
Parts:
- added C?: 560pF 250v, Capacitors_SMD:C_0603, symbol C
- added C?: 1nF, Capacitors_SMD:C_0805, symbol C
- added C?: 220pF, Capacitors_SMD:C_0805, symbol C
- added C?: 430pF, Capacitors_SMD:C_0805, symbol C
- added C? (x2): 1uF 250v, Capacitors_SMD:C_1812_HandSoldering, symbol C
- added C?: 100pF 250v, Capacitors_SMD:C_0805, symbol C
- added C? (x2): 100uF 16v, Capacitors_SMD:C_1210, symbol C
- added C?: 0.1uF 16v, Capacitors_SMD:C_0805, symbol C
- added C? (x2): 0.1uF 250v, Capacitors_SMD:C_0805, symbol C
- added C?: 0.1uF, Capacitors_SMD:C_0805, symbol C
- added C?: 47uF 16v, Capacitors_SMD:C_1210, symbol C
- added C? (x6): 0.1uF, symbol C
- added D?: ES1D, Diodes_SMD:D_SMA, symbol D
- added D?: BAT54, Diodes_SMD:D_SOD-323_HandSoldering, symbol D_Schottky
- added L?: 33uH, NixieSupply5vto160vDCMBoost_socket:Choke_SMD_12x12mm_Wurth_WE-PD, symbol L
- added L? (x2): 60ohm 100Mhz, Resistors_SMD:R_0805, symbol L
- added NE? (x4): Lamp_Neon, symbol Lamp_Neon
- added P?: USB_OTG, NixieSupply5vto160vDCMBoost_socket:USB_Micro-B_Wurth_3A_Non-OVAL-Drill, symbol USB_OTG
- added Q?: FDS2672CT, etaclock:SOIC-8-N, symbol FDMS86255ET150
- added Q?: MMBTA42, TO_SOT_Packages_SMD:SOT-23, symbol MMBT3904
- added R? (x2): 15k, symbol R
- added R?: 0.1 1/2W, Resistors_SMD:R_0805, symbol R
- added R? (x2): 1k, Resistors_SMD:R_0805, symbol R
- added R?: 634k, Resistors_SMD:R_0805, symbol R
- added R?: 7.68k, Resistors_SMD:R_0805, symbol R
- added R?: 0 Ohm, Resistors_SMD:R_0805, symbol R
- added R?: N.U., Resistors_SMD:R_0805, symbol R
- added R?: 60.4k, Resistors_SMD:R_0805, symbol R
- added R?: 4.12k, Resistors_SMD:R_0805, symbol R
- added R?: 2k, Resistors_SMD:R_0805, symbol R
- added R? (x2): 100k, Resistors_SMD:R_0805, symbol R
- added U?: UCC3803, NixieSupply5vto160vDCMBoost_socket:SOIC-8-N, symbol AAC243
Connections:
- net 1h8: no longer U?.18 (HVo28)
- net 1h9: no longer U?.19 (HVo29)
- net GND: now also C?.2, C?.2, C?.2, C?.2, C?.2, C?.2, C?.2, C?.2, C?.2, C?.2, C?.2, C?.2, P?.5 (GND), P?.6 (Shield), Q?.2 (E), R?.1, R?.2, R?.2, U?.5 (GND); no longer U?.30 (GND)
- net +5V: now reaches U?.31 (VDD)
- net +5V: now also LED?.1 (VDD), LED?.1 (VDD), LED?.1 (VDD), LED?.1 (VDD), LED?.1 (VDD), LED?.1 (VDD), U?.31 (VDD), C?.1, C?.1, C?.1, C?.1, C?.1, C?.1
- net at U?.33 (DataIN): now also U?.23 (DataOut)
- net VSS: now reaches LED?.3 (VSS)
- net VSS: now also LED?.3 (VSS), LED?.3 (VSS), LED?.3 (VSS), LED?.3 (VSS), LED?.3 (VSS), C?.2, C?.2, C?.2, C?.2, C?.2, C?.2
- net SPI: now reaches LED?.4 (DIN)
- net VDDA renamed +160V
- net +160V: now also C?.1, L?.1, R?.1, R?.2
- new net: NE?.1, NE?.2 (x2)
- new net: NE?.1, R?.2
- new net: NE?.1, R?.1
- new net: C?.1, C?.1, C?.1, C?.1, D?.1 (K), L?.2, R?.1
- new net: C?.1, D?.2 (A), L?.1, Q?.5 (D), Q?.6 (D), Q?.7 (D), Q?.8 (D)
- new net: C?.1, L?.1, L?.2, U?.7 (Vcc)
- new net: Q?.1 (S), Q?.2 (S), Q?.3 (S), R?.1, R?.1
- new net: C?.1, D?.2 (A), R?.2, U?.1 (COMP)
- new net: C?.2, R?.1, R?.1, R?.1, R?.2, U?.2 (FB)
- new net: C?.1, R?.1, R?.2, U?.3 (Isense)
- new net: C?.1, R?.1, U?.4 (R/C)
- new net: Q?.4 (G), U?.6 (OUT)
- new net: C?.1, R?.2, R?.2, U?.8 (Vref)
- new net: C?.2, R?.2
- new net: C?.1, D?.1 (K), Q?.3 (C), R?.1, R?.2
- new net: Q?.1 (B), R?.1, R?.1
- new net 5v_Power: C?.1, C?.1, L?.2, P?.1 (VBUS), R?.2, R?.2
- new net HM: NE?.2, U?.19 (HVo29)
- new net MS: NE?.2, U?.18 (HVo28)
- new net N_ENABLE: R?.2
- no-connect marks 0 -> 1
Other:
- note added: "OUTPUT SET to 167Volts"
- moved on the sheet: J?, LED?, NX?, R?, U?
